Commit message: update 1/7

File: src/mybot_description/urdf/mybot.gazebo.urdf (robot description, URDF)
Before this commit: robot mybot, 6 links, 5 joints
Links:
- added link base_footprint
- added link lidar_link, mass 0.1; collision cylinder length=0.1 radius=0.03; visual cylinder length=0.1 radius=0.03
Joints:
- added joint base_joint: type fixed, parent base_footprint, child base_link, origin xyz=0 0 0.2352 rpy=0 0 0
- added joint lidar_joint: type fixed, parent base_link, child lidar_link, origin xyz=0 0 0.13 rpy=0 0 0

File: src/mybot_description/urdf/mybot.urdf (robot description, URDF)
Before this commit: robot mybot, 6 links, 5 joints
Links:
- added link base_footprint
Joints:
- added joint base_joint: type fixed, parent base_footprint, child base_link, origin xyz=0 0 0 rpy=0 0 0
