Commit message: add 1/9

File: src/mybot_description/urdf/mybot.gazebo2.xacro (robot description, xacro)
@@ -23,5 +23,5 @@
         <mu1>${base_mu1}</mu1>
         <mu2>${base_mu2}</mu2>
-        <material>Gazebo/Grey</material>
+        <!-- <material>Gazebo/Grey</material> -->
     </gazebo>
     <gazebo reference="camera_link">
