Commit message: add 1/16 update

File: src/mybot_description/urdf/mybot.gazebo.xacro (robot description, xacro)
@@ -86,35 +86,36 @@
     <gazebo reference="lidar_link">
         <sensor type="ray" name="lidar_sensor">
-        <pose>0 0 0 0 0 0</pose>
-        <visualize>true</visualize>
-        <update_rate>10</update_rate>
-        <ray>
-            <scan>
-            <horizontal>
-                <samples>360</samples>
-                <resolution>1</resolution>
-                <min_angle>-3.14159</min_angle>
-                <max_angle>3.14159</max_angle>
-            </horizontal>
-            </scan>
-            <range>
-                <min>0.10</min>
-                <max>10.0</max>
-                <resolution>0.01</resolution>
-            </range>
-            <noise>
-                <type>gaussian</type>
-                <mean>0.0</mean>
-                <stddev>0.01</stddev>
-            </noise>
-        </ray>
-        <plugin name="lidar_controller" filename="libgazebo_ros_ray_sensor.so">
-            <ros>
-                <namespace>/</namespace>
-                <remapping>~/out:=scan</remapping>
-            </ros>
-            <output_type>sensor_msgs/LaserScan</output_type>
-            <frame_name>lidar_link</frame_name>
-        </plugin>
+            <always_on>true</always_on>
+            <visualize>false</visualize>
+            <pose>0 0 0 0 0 0</pose>
+            <update_rate>10</update_rate>
+            <ray>
+                <scan>
+                    <horizontal>
+                        <samples>360</samples>
+                        <resolution>1</resolution>
+                        <min_angle>-3.14159</min_angle>
+                        <max_angle>3.14159</max_angle>
+                    </horizontal>
+                </scan>
+                <range>
+                    <min>0.10</min>
+                    <max>10.0</max>
+                    <resolution>0.01</resolution>
+                </range>
+                <noise>
+                    <type>gaussian</type>
+                    <mean>0.0</mean>
+                    <stddev>0.01</stddev>
+                </noise>
+            </ray>
+            <plugin name="lidar_controller" filename="libgazebo_ros_ray_sensor.so">
+                <ros>
+                    <!-- <namespace>/</namespace> -->
+                    <remapping>~/out:=scan</remapping>
+                </ros>
+                <output_type>sensor_msgs/LaserScan</output_type>
+                <frame_name>lidar_link</frame_name>
+            </plugin>
         </sensor>
     </gazebo>
@@ -122,27 +123,41 @@
     <gazebo reference="camera_link">
         <sensor type="camera" name="camera_sensor">
-        <update_rate>${update_rate}</update_rate>
-        <camera name="camera">
-            <horizontal_fov>1.3962634</horizontal_fov>
-            <image>
-            <width>640</width>
-            <height>480</height>
-            <format>R8G8B8</format>
-            </image>
-            <clip>
-            <near>0.02</near>
-            <far>300</far>
-            </clip>
-        </camera>
-        <plugin name="camera_controller" filename="libgazebo_ros_camera.so">
-            <ros>
-                <namespace>/</namespace>
-                <remapping>camera/image_raw:=camera/image</remapping>
-                <remapping>camera/camera_info:=camera/camera_info</remapping>
-            </ros>
-            <camera_name>camera</camera_name>
-            <frame_name>camera_link</frame_name>
-            <hack_baseline>0.07</hack_baseline>
-        </plugin>
+            <always_on>true</always_on>
+            <visualize>true</visualize>
+            <update_rate>${update_rate}</update_rate>
+            <camera name="camera">
+                <horizontal_fov>1.3962634</horizontal_fov>
+                <image>
+                    <width>640</width>
+                    <height>480</height>
+                    <format>R8G8B8</format>
+                </image>
+                <clip>
+                    <near>0.02</near>
+                    <far>300</far>
+                </clip>
+                <!-- <lens>
+                    <type>custom</type>
+                    <custom_function>
+                        <c1>1.05</c1>
+                        <c2>4</c2>
+                        <f>1.0</f>
+                        <fun>tan</fun>
+                    </custom_function>
+                    <scale_to_hfov>true</scale_to_hfov>
+                    <cutoff_angle>3.1415</cutoff_angle>
+                    <env_texture_size>512</env_texture_size>
+                </lens> -->
+            </camera>
+                <plugin name="camera_controller" filename="libgazebo_ros_camera.so">
+                    <ros>
+                        <namespace>/</namespace>
+                        <remapping>camera/image_raw:=camera/image</remapping>
+                        <remapping>camera/camera_info:=camera/camera_info</remapping>
+                    </ros>
+                    <camera_name>camera</camera_name>
+                    <frame_name>camera_link</frame_name>
+                    <hack_baseline>0.07</hack_baseline>
+                </plugin>
         </sensor>
     </gazebo>

File: src/mybot_description/urdf/mybot.gazebo2.xacro (robot description, xacro)
@@ -85,10 +85,10 @@
                     <resolution>0.01</resolution> -->
                 </range>
-                <!-- 가상의 노이즈 추가
+                <!-- 가상의 노이즈 추가 -->
                 <noise>
                     <type>gaussian</type>
                     <mean>0.0</mean>
                     <stddev>0.01</stddev>
-                </noise> -->
+                </noise>
             </ray>
             <plugin name="lidar_controller" filename="libgazebo_ros_ray_sensor.so">

File: src/mybot_description/urdf/mybot2.xacro (robot description, xacro)
@@ -1,20 +1,24 @@
 <?xml version="1.0"?>
 <robot name="mybot" xmlns:xacro="http://www.ros.org/wiki/xacro">
-  <xacro:include filename="$(find mybot_description)/urdf/mybot.gazebo2.xacro"/>
-  <xacro:property name="base_mass"   value="50.0"/>
-  <xacro:property name="base_width"  value="0.38"/>
+  <!-- Gazebo 설정 파일 포함 -->
+  <xacro:include filename="$(find mybot_description)/urdf/mybot.gazebo.xacro"/>
+  <!-- Properties (변수) 정의 -->
+  <xacro:property name="base_mass" value="50.0"/>
+  <xacro:property name="base_width" value="0.38"/>
   <xacro:property name="base_length" value="0.925"/>
   <xacro:property name="base_height" value="0.21"/>
-  <xacro:property name="wheel_mass"   value="8.0"/>
   <xacro:property name="wheel_radius" value="0.16459"/>
   <xacro:property name="wheel_length" value="0.11653"/>
+  <xacro:property name="wheel_mass" value="8.0"/>
   <xacro:property name="wheel_offset_x" value="0.249"/>
   <xacro:property name="wheel_offset_y" value="0.29153"/>
   <xacro:property name="wheel_offset_z" value="-0.0702"/>
-  <xacro:property name="camera_size"   value="0.02"/>
-  <xacro:property name="lidar_radius"  value="0.03"/>
-  <xacro:property name="lidar_length"  value="0.1"/>
+  <xacro:property name="camera_size" value="0.02"/>
+  <xacro:property name="lidar_radius" value="0.03"/>
+  <xacro:property name="lidar_length" value="0.1"/>
+  <!-- 재질 정의 -->
   <material name="red"><color rgba="1.0 0.0 0.0 1.0"/></material>
   <material name="black"><color rgba="0 0 0 1"/></material>
+  <!-- 바퀴 매크로 정의 -->
   <xacro:macro name="wheel" params="prefix wheel_type *origin *axis">
     <link name="${prefix}_wheel_link">
@@ -24,5 +28,7 @@
       <collision>
         <origin rpy="1.570795 0 0" xyz="0 0 0"/>
-        <geometry><cylinder length="${wheel_length}" radius="${wheel_radius}"/></geometry>
+        <geometry>
+          <cylinder length="${wheel_length}" radius="${wheel_radius}"/>
+        </geometry>
       </collision>
       <inertial>
@@ -42,6 +48,8 @@
       <dynamics damping="0.0" friction="20"/>
     </joint>
+    <!-- Gazebo 속성 적용 -->
     <xacro:wheel_gazebo prefix="${prefix}"/>
   </xacro:macro>
+  <!-- 바퀴 생성 -->
   <xacro:wheel prefix="front_right" wheel_type="wheel_type1">
     <origin rpy="3.14 0 0" xyz="${wheel_offset_x} ${-wheel_offset_y} ${wheel_offset_z}"/>
@@ -60,5 +68,7 @@
     <axis xyz="0 -1 0"/>
   </xacro:wheel>
+  <!-- Base footprint link -->
   <link name="base_footprint"/>
+  <!-- Base link -->
   <link name="base_link">
     <visual>
@@ -68,9 +78,13 @@
     <collision>
       <origin xyz="0 0 0.008"/>
-      <geometry><box size="${base_length} ${base_width} ${base_height}"/></geometry>
+      <geometry>
+        <box size="${base_length} ${base_width} ${base_height}"/>
+      </geometry>
     </collision>
     <collision>
       <origin xyz="0 0 0.035"/>
-      <geometry><box size="0.154 0.627 0.07"/></geometry>
+      <geometry>
+        <box size="0.154 0.627 0.07"/>
+      </geometry>
     </collision>
     <inertial>
@@ -87,11 +101,16 @@
     <origin xyz="0 0 0.2352" rpy="0 0 0"/>
   </joint>
+  <!-- Camera link -->
   <link name="camera_link">
     <visual>
-      <geometry><box size="${camera_size} ${camera_size} ${camera_size}"/></geometry>
+      <geometry>
+        <box size="${camera_size} ${camera_size} ${camera_size}"/>
+      </geometry>
       <material name="red"/>
     </visual>
     <collision>
-      <geometry><box size="${camera_size} ${camera_size} ${camera_size}"/></geometry>
+      <geometry>
+        <box size="${camera_size} ${camera_size} ${camera_size}"/>
+      </geometry>
     </collision>
     <inertial>
@@ -103,13 +122,20 @@
   </link>
   <joint name="camera_joint" type="fixed">
-    <parent link="base_link"/><child link="camera_link"/><origin xyz="0.40 0.0 0.04"/>
+    <parent link="base_link"/>
+    <child link="camera_link"/>
+    <origin xyz="0.40 0.0 0.04"/>
   </joint>
+  <!-- 2D LiDAR Link -->
   <link name="lidar_link">
     <visual>
-      <geometry><cylinder radius="${lidar_radius}" length="${lidar_length}"/></geometry>
+      <geometry>
+        <cylinder radius="${lidar_radius}" length="${lidar_length}"/>
+      </geometry>
       <material name="black"/>
     </visual>
     <collision>
-      <geometry><cylinder radius="${lidar_radius}" length="${lidar_length}"/></geometry>
+      <geometry>
+        <cylinder radius="${lidar_radius}" length="${lidar_length}"/>
+      </geometry>
     </collision>
     <inertial>
@@ -117,9 +143,11 @@
       <inertia ixx="${(1/12) * 0.1 * (3*lidar_radius*lidar_radius + lidar_length*lidar_length)}" ixy="0" ixz="0"
                iyy="${(1/12) * 0.1 * (3*lidar_radius*lidar_radius + lidar_length*lidar_length)}" iyz="0"
-               izz="${(1/2) * 0.1 * lidar_radius*lidar_radius}"/>
+                 izz="${(1/2) * 0.1 * (lidar_radius*lidar_radius)}"/>
     </inertial>
   </link>
   <joint name="lidar_joint" type="fixed">
-    <parent link="base_link"/><child link="lidar_link"/><origin xyz="0 0 0.13" rpy="0 0 0"/>
+    <parent link="base_link"/>
+    <child link="lidar_link"/>
+    <origin xyz="0 0 0.13" rpy="0 0 0"/>
   </joint>
 </robot>

File: src/mybot_description/urdf/mybot3_cam.xacro (robot description, xacro)
@@ -1,7 +1,7 @@
 <?xml version="1.0"?>
 <robot name="mybot" xmlns:xacro="http://www.ros.org/wiki/xacro">
-  <!-- Gazebo 설정 파일 포함 -->
+  <xacro:include filename="$(find realsense2_description)/urdf/_d435i.urdf.xacro"/>
   <xacro:include filename="$(find mybot_description)/urdf/mybot.gazebo.xacro"/>
-  <!-- Properties (변수) 정의 -->
+  <xacro:property name="base_mass" value="50.0"/>
   <xacro:property name="base_width" value="0.38"/>
   <xacro:property name="base_length" value="0.925"/>
@@ -13,15 +13,9 @@
   <xacro:property name="wheel_offset_y" value="0.29153"/>
   <xacro:property name="wheel_offset_z" value="-0.0702"/>
-  <xacro:property name="camera_size" value="0.02"/>
   <xacro:property name="lidar_radius" value="0.03"/>
   <xacro:property name="lidar_length" value="0.1"/>
-  <!-- 계산된 속성
-  <xacro:property name="wheel_separation" value="${wheel_offset_y * 2}"/>
-  -->
-  <!-- 재질 정의 -->
-  <material name="red"><color rgba="1.0 0.0 0.0 1.0"/></material>
-  <material name="black"><color rgba="0 0 0 1"/></material>
-  <!-- 바퀴 매크로 정의 -->
-  <xacro:macro name="wheel" params="prefix pos_x pos_y pos_z flip wheel_type *origin *axis">
+  <material name="red">  <color rgba="1.0 0.0 0.0 1.0"/></material>
+  <material name="black"><color rgba="0.0 0.0 0.0 0.8"/></material>
+  <xacro:macro name="wheel" params="prefix wheel_type *origin *axis">
     <link name="${prefix}_wheel_link">
       <visual>
@@ -29,5 +23,5 @@
       </visual>
       <collision>
-        <origin rpy="1.570795 0 0"/>
+        <origin rpy="1.570795 0 0" xyz="0 0 0"/>
         <geometry>
           <cylinder length="${wheel_length}" radius="${wheel_radius}"/>
@@ -35,12 +29,11 @@
       </collision>
       <inertial>
+        <origin xyz="0 0 0" rpy="0 0 0"/>
         <mass value="${wheel_mass}"/>
         <inertia ixx="${(1/12) * wheel_mass * (3*wheel_radius*wheel_radius + wheel_length*wheel_length)}" ixy="0" ixz="0"
-                 iyy="${(1/12) * wheel_mass * (3*wheel_radius*wheel_radius + wheel_length*wheel_length)}" iyz="0"
-                 izz="${(1/2) * wheel_mass * (wheel_radius*wheel_radius)}"/>
-        <!-- <inertia ixx="0.1171" ixy="0" ixz="0" iyy="0.1361" iyz="0" izz="0.1171"/> -->
+                iyy="${(1/12) * wheel_mass * (3*wheel_radius*wheel_radius + wheel_length*wheel_length)}" iyz="0"
+                izz="${(1/2) * wheel_mass * (wheel_radius*wheel_radius)}"/>
       </inertial>
     </link>
-    <!--바퀴 joint는 diff_drvie 플러그 연동됨으로 확인 필요함-->
     <joint name="${prefix}_wheel" type="continuous">
       <parent link="base_link"/>
@@ -50,27 +43,23 @@
       <dynamics damping="0.0" friction="20"/>
     </joint>
-    <!-- Gazebo 속성 적용 -->
     <xacro:wheel_gazebo prefix="${prefix}"/>
   </xacro:macro>
-  <!-- 바퀴 생성 -->
-  <xacro:wheel prefix="front_right" pos_x="${wheel_offset_x}" pos_y="${-wheel_offset_y}" pos_z="${wheel_offset_z}" flip="true" wheel_type="wheel_type1">
+  <xacro:wheel prefix="front_right" wheel_type="wheel_type1">
     <origin rpy="3.14 0 0" xyz="${wheel_offset_x} ${-wheel_offset_y} ${wheel_offset_z}"/>
     <axis xyz="0 -1 0"/>
   </xacro:wheel>
-  <xacro:wheel prefix="front_left" pos_x="${wheel_offset_x}" pos_y="${wheel_offset_y}" pos_z="${wheel_offset_z}" flip="false" wheel_type="wheel_type2">
+  <xacro:wheel prefix="front_left" wheel_type="wheel_type2">
     <origin rpy="0 0 0" xyz="${wheel_offset_x} ${wheel_offset_y} ${wheel_offset_z}"/>
     <axis xyz="0 1 0"/>
   </xacro:wheel>
-  <xacro:wheel prefix="rear_left" pos_x="${-wheel_offset_x}" pos_y="${wheel_offset_y}" pos_z="${wheel_offset_z}" flip="false" wheel_type="wheel_type2">
+  <xacro:wheel prefix="rear_left" wheel_type="wheel_type2">
     <origin rpy="0 0 0" xyz="${-wheel_offset_x} ${wheel_offset_y} ${wheel_offset_z}"/>
     <axis xyz="0 1 0"/>
   </xacro:wheel>
-  <xacro:wheel prefix="rear_right" pos_x="${-wheel_offset_x}" pos_y="${-wheel_offset_y}" pos_z="${wheel_offset_z}" flip="true" wheel_type="wheel_type1">
+  <xacro:wheel prefix="rear_right" wheel_type="wheel_type1">
     <origin rpy="3.14 0 0" xyz="${-wheel_offset_x} ${-wheel_offset_y} ${wheel_offset_z}"/>
     <axis xyz="0 -1 0"/>
   </xacro:wheel>
-  <!-- Base footprint link -->
   <link name="base_footprint"/>
-  <!-- Base link -->
   <link name="base_link">
     <visual>
@@ -91,10 +80,9 @@
     </collision>
     <inertial>
-      <mass value="50"/>
+      <mass value="${base_mass}"/>
       <origin xyz="0.0 0.0 0.015"/>
-      <!-- <inertia ixx="2.288641" ixy="0" ixz="0" iyy="5.103976" iyz="0" izz="3.431465"/></inertial> -->
-      <inertia ixx="${(1/12) * 50 * (base_width*base_width + base_height*base_height)}" ixy="0" ixz="0"
-             iyy="${(1/12) * 50 * (base_length*base_length + base_height*base_height)}" iyz="0"
-             izz="${(1/12) * 50 * (base_length*base_length + base_width*base_width)}"/>
+      <inertia ixx="${(1/12) * base_mass * (base_width*base_width + base_height*base_height)}" ixy="0" ixz="0"
+               iyy="${(1/12) * base_mass * (base_length*base_length + base_height*base_height)}" iyz="0"
+               izz="${(1/12) * base_mass * (base_length*base_length + base_width*base_width)}"/>
     </inertial>
   </link>
@@ -104,31 +92,7 @@
     <origin xyz="0 0 0.2352" rpy="0 0 0"/>
   </joint>
-  <!-- Camera link -->
-  <link name="camera_link">
-    <visual>
-      <geometry>
-        <box size="${camera_size} ${camera_size} ${camera_size}"/>
-      </geometry>
-      <material name="red"/>
-    </visual>
-    <collision>
-      <geometry>
-        <box size="${camera_size} ${camera_size} ${camera_size}"/>
-      </geometry>
-    </collision>
-    <inertial>
-      <mass value="0.1"/>
-      <!-- <inertia ixx="0.000083" ixy="0" ixz="0" iyy="0.000083" iyz="0" izz="0.000083"/></inertial> -->
-      <inertia ixx="${(1/12) * 0.1 * (camera_size*camera_size + camera_size*camera_size)}" ixy="0" ixz="0"
-             iyy="${(1/12) * 0.1 * (camera_size*camera_size + camera_size*camera_size)}" iyz="0"
-             izz="${(1/12) * 0.1 * (camera_size*camera_size + camera_size*camera_size)}"/>
-    </inertial>
-  </link>
-  <joint name="camera_joint" type="fixed">
-    <parent link="base_link"/>
-    <child link="camera_link"/>
-    <origin xyz="0.40 0.0 0.04"/>
-  </joint>
-  <!-- 2D LiDAR Link -->
+  <xacro:sensor_d435i parent="base_link" name="camera" use_nominal_extrinsics="true">
+    <origin xyz="0.40 0.0 0.04" rpy="0 0 0"/>
+  </xacro:sensor_d435i>
   <link name="lidar_link">
     <visual>
@@ -145,9 +109,8 @@
     <inertial>
       <mass value="0.1"/>
-      <!-- <inertia ixx="0.000045" ixy="0" ixz="0" iyy="0.000045" iyz="0" izz="0.000075"/></inertial> -->
       <inertia ixx="${(1/12) * 0.1 * (3*lidar_radius*lidar_radius + lidar_length*lidar_length)}" ixy="0" ixz="0"
-                 iyy="${(1/12) * 0.1 * (3*lidar_radius*lidar_radius + lidar_length*lidar_length)}" iyz="0"
-                 izz="${(1/2) * 0.1 * (lidar_radius*lidar_radius)}"/>
-      </inertial>
+              iyy="${(1/12) * 0.1 * (3*lidar_radius*lidar_radius + lidar_length*lidar_length)}" iyz="0"
+              izz="${(1/2) * 0.1 * (lidar_radius*lidar_radius)}"/>
+    </inertial>
   </link>
   <joint name="lidar_joint" type="fixed">
