Commit message: add 1/16 update

File: src/mybot_description/urdf/mybot_cam.xacro (robot description, xacro)
@@ -3,5 +3,9 @@
   <!-- Gazebo 설정 파일 포함 -->
   <xacro:include filename="$(find mybot_description)/urdf/mybot.gazebo.xacro"/>
+  <xacro:include filename="$(find realsense2_description)/urdf/_d435i.urdf.xacro" />
+  <!-- <xacro:include filename="/home/won/etc_ws/src/realsense-ros/realsense2_description/urdf/_d435i.urdf.xacro"/> -->
+  <xacro:include filename="/home/won/etc_ws/install/realsense2_description/share/realsense2_description/urdf/_d435i.urdf.xacro" />
   <!-- Properties (변수) 정의 -->
+  <xacro:property name="base_mass" value="50.0"/>
   <xacro:property name="base_width" value="0.38"/>
   <xacro:property name="base_length" value="0.925"/>
@@ -16,12 +20,9 @@
   <xacro:property name="lidar_radius" value="0.03"/>
   <xacro:property name="lidar_length" value="0.1"/>
-  <!-- 계산된 속성
-  <xacro:property name="wheel_separation" value="${wheel_offset_y * 2}"/>
-  -->
   <!-- 재질 정의 -->
   <material name="red"><color rgba="1.0 0.0 0.0 1.0"/></material>
   <material name="black"><color rgba="0 0 0 1"/></material>
   <!-- 바퀴 매크로 정의 -->
-  <xacro:macro name="wheel" params="prefix pos_x pos_y pos_z flip wheel_type *origin *axis">
+  <xacro:macro name="wheel" params="prefix wheel_type *origin *axis">
     <link name="${prefix}_wheel_link">
       <visual>
@@ -29,5 +30,5 @@
       </visual>
       <collision>
-        <origin rpy="1.570795 0 0"/>
+        <origin rpy="1.570795 0 0" xyz="0 0 0"/>
         <geometry>
           <cylinder length="${wheel_length}" radius="${wheel_radius}"/>
@@ -35,9 +36,9 @@
       </collision>
       <inertial>
+        <origin xyz="0 0 0" rpy="0 0 0"/>
         <mass value="${wheel_mass}"/>
         <inertia ixx="${(1/12) * wheel_mass * (3*wheel_radius*wheel_radius + wheel_length*wheel_length)}" ixy="0" ixz="0"
                  iyy="${(1/12) * wheel_mass * (3*wheel_radius*wheel_radius + wheel_length*wheel_length)}" iyz="0"
                  izz="${(1/2) * wheel_mass * (wheel_radius*wheel_radius)}"/>
-        <!-- <inertia ixx="0.1171" ixy="0" ixz="0" iyy="0.1361" iyz="0" izz="0.1171"/> -->
       </inertial>
     </link>
@@ -54,17 +55,17 @@
   </xacro:macro>
   <!-- 바퀴 생성 -->
-  <xacro:wheel prefix="front_right" pos_x="${wheel_offset_x}" pos_y="${-wheel_offset_y}" pos_z="${wheel_offset_z}" flip="true" wheel_type="wheel_type1">
+  <xacro:wheel prefix="front_right" wheel_type="wheel_type1">
     <origin rpy="3.14 0 0" xyz="${wheel_offset_x} ${-wheel_offset_y} ${wheel_offset_z}"/>
     <axis xyz="0 -1 0"/>
   </xacro:wheel>
-  <xacro:wheel prefix="front_left" pos_x="${wheel_offset_x}" pos_y="${wheel_offset_y}" pos_z="${wheel_offset_z}" flip="false" wheel_type="wheel_type2">
+  <xacro:wheel prefix="front_left" wheel_type="wheel_type2">
     <origin rpy="0 0 0" xyz="${wheel_offset_x} ${wheel_offset_y} ${wheel_offset_z}"/>
     <axis xyz="0 1 0"/>
   </xacro:wheel>
-  <xacro:wheel prefix="rear_left" pos_x="${-wheel_offset_x}" pos_y="${wheel_offset_y}" pos_z="${wheel_offset_z}" flip="false" wheel_type="wheel_type2">
+  <xacro:wheel prefix="rear_left" wheel_type="wheel_type2">
     <origin rpy="0 0 0" xyz="${-wheel_offset_x} ${wheel_offset_y} ${wheel_offset_z}"/>
     <axis xyz="0 1 0"/>
   </xacro:wheel>
-  <xacro:wheel prefix="rear_right" pos_x="${-wheel_offset_x}" pos_y="${-wheel_offset_y}" pos_z="${wheel_offset_z}" flip="true" wheel_type="wheel_type1">
+  <xacro:wheel prefix="rear_right" wheel_type="wheel_type1">
     <origin rpy="3.14 0 0" xyz="${-wheel_offset_x} ${-wheel_offset_y} ${wheel_offset_z}"/>
     <axis xyz="0 -1 0"/>
@@ -91,10 +92,9 @@
     </collision>
     <inertial>
-      <mass value="50"/>
+      <mass value="${base_mass}"/>
       <origin xyz="0.0 0.0 0.015"/>
-      <!-- <inertia ixx="2.288641" ixy="0" ixz="0" iyy="5.103976" iyz="0" izz="3.431465"/></inertial> -->
-      <inertia ixx="${(1/12) * 50 * (base_width*base_width + base_height*base_height)}" ixy="0" ixz="0"
-             iyy="${(1/12) * 50 * (base_length*base_length + base_height*base_height)}" iyz="0"
-             izz="${(1/12) * 50 * (base_length*base_length + base_width*base_width)}"/>
+      <inertia ixx="${(1/12) * base_mass * (base_width*base_width + base_height*base_height)}" ixy="0" ixz="0"
+               iyy="${(1/12) * base_mass * (base_length*base_length + base_height*base_height)}" iyz="0"
+               izz="${(1/12) * base_mass * (base_length*base_length + base_width*base_width)}"/>
     </inertial>
   </link>
@@ -119,8 +119,7 @@
     <inertial>
       <mass value="0.1"/>
-      <!-- <inertia ixx="0.000083" ixy="0" ixz="0" iyy="0.000083" iyz="0" izz="0.000083"/></inertial> -->
       <inertia ixx="${(1/12) * 0.1 * (camera_size*camera_size + camera_size*camera_size)}" ixy="0" ixz="0"
-             iyy="${(1/12) * 0.1 * (camera_size*camera_size + camera_size*camera_size)}" iyz="0"
-             izz="${(1/12) * 0.1 * (camera_size*camera_size + camera_size*camera_size)}"/>
+               iyy="${(1/12) * 0.1 * (camera_size*camera_size + camera_size*camera_size)}" iyz="0"
+               izz="${(1/12) * 0.1 * (camera_size*camera_size + camera_size*camera_size)}"/>
     </inertial>
   </link>
@@ -145,9 +144,8 @@
     <inertial>
       <mass value="0.1"/>
-      <!-- <inertia ixx="0.000045" ixy="0" ixz="0" iyy="0.000045" iyz="0" izz="0.000075"/></inertial> -->
       <inertia ixx="${(1/12) * 0.1 * (3*lidar_radius*lidar_radius + lidar_length*lidar_length)}" ixy="0" ixz="0"
-                 iyy="${(1/12) * 0.1 * (3*lidar_radius*lidar_radius + lidar_length*lidar_length)}" iyz="0"
+               iyy="${(1/12) * 0.1 * (3*lidar_radius*lidar_radius + lidar_length*lidar_length)}" iyz="0"
                  izz="${(1/2) * 0.1 * (lidar_radius*lidar_radius)}"/>
-      </inertial>
+    </inertial>
   </link>
   <joint name="lidar_joint" type="fixed">
