Commit message: add simulation

File: src/cybertruck_description/urdf/cybertruck.urdf (robot description, URDF)
Before this commit: robot cybertruck, 5 links, 4 joints
Joints:
- joint rear_left_wheel: origin xyz=-1.97228 0.91457 -0.66346 rpy=1.57080 -0.00000 3.14159 -> xyz=-1.97228 0.91457 -0.66346 rpy=1.57080 0.00000 3.14159

Commit message: add 1/8

File: src/cybertruck_description/urdf/cybertruck.urdf (robot description, URDF)
Before this commit: robot cybertruck, 5 links, 4 joints
Links:
- added link base_footprint
Joints:
- added joint base_joint: type fixed, parent base_footprint, child base_link, origin xyz=0 0 0.2352 rpy=0 0 0

File: src/mybot_description/urdf/mybot.gazebo.xacro (robot description, xacro)
@@ -19,9 +19,9 @@
         </gazebo>
     </xacro:macro>
-    <!-- 각 바퀴에 Gazebo 속성 적용 -->
+    <!-- 각 바퀴에 Gazebo 속성 적용
     <xacro:wheel_gazebo prefix="front_right"/>
     <xacro:wheel_gazebo prefix="front_left"/>
     <xacro:wheel_gazebo prefix="rear_left"/>
-    <xacro:wheel_gazebo prefix="rear_right"/>
+    <xacro:wheel_gazebo prefix="rear_right"/> -->
     <!-- Gazebo 속성: 베이스 링크 -->
     <gazebo reference="base_link">
@@ -137,7 +137,7 @@
         <plugin name="camera_controller" filename="libgazebo_ros_camera.so">
             <ros>
-            <namespace>/</namespace>
-            <remapping>camera/image_raw:=camera/image</remapping>
-            <remapping>camera/camera_info:=camera/camera_info</remapping>
+                <namespace>/</namespace>
+                <remapping>camera/image_raw:=camera/image</remapping>
+                <remapping>camera/camera_info:=camera/camera_info</remapping>
             </ros>
             <camera_name>camera</camera_name>

File: src/mybot_description/urdf/mybot.urdf (robot description, URDF)
Before this commit: robot mybot, 7 links, 6 joints
Links:
- added link lidar_link, mass 0.1; collision cylinder length=0.1 radius=0.03; visual cylinder length=0.1 radius=0.03
- link base_link: mass None -> 50; geometry collision box size=0.154 0.627 0.07; collision box size=0.925 0.38 0.21
- link camera_link: mass None -> 0.1; geometry collision box size=0.02 0.02 0.02; visual box size=0.02 0.02 0.02
- link front_left_wheel_link: mass None -> 8; geometry collision cylinder length=0.11653 radius=0.16459; visual mesh filename=package://mybot_description/meshes/wheel_type2.dae
- link front_right_wheel_link: mass None -> 8; geometry collision cylinder length=0.11653 radius=0.16459; visual mesh filename=package://mybot_description/meshes/wheel_type1.dae
- link rear_left_wheel_link: mass None -> 8; geometry collision cylinder length=0.11653 radius=0.16459; visual mesh filename=package://mybot_description/meshes/wheel_type2.dae
- link rear_right_wheel_link: mass None -> 8; geometry collision cylinder length=0.11653 radius=0.16459; visual mesh filename=package://mybot_description/meshes/wheel_type1.dae
Joints:
- added joint lidar_joint: type fixed, parent base_link, child lidar_link, origin xyz=0 0 0.13 rpy=0 0 0
- joint base_joint: origin xyz=0 0 0 rpy=0 0 0 -> xyz=0 0 0.2352 rpy=0 0 0

File: src/mybot_description/urdf/mybot2.xacro (robot description, xacro)
@@ -1,28 +1,21 @@
 <?xml version="1.0"?>
-<robot name="mybot"
-  xmlns:xacro="http://www.ros.org/wiki/xacro">
-  <!-- Gazebo 설정 파일 포함 -->
-  <xacro:include filename="$(find mybot_description)/urdf/mybot.gazebo.xacro"/>
-  <!-- Properties (변수) 정의 -->
-  <xacro:property name="base_width" value="0.38"/>
+<robot name="mybot" xmlns:xacro="http://www.ros.org/wiki/xacro">
+  <xacro:include filename="$(find mybot_description)/urdf/mybot.gazebo2.xacro"/>
+  <xacro:property name="base_mass"   value="50.0"/>
+  <xacro:property name="base_width"  value="0.38"/>
   <xacro:property name="base_length" value="0.925"/>
   <xacro:property name="base_height" value="0.21"/>
+  <xacro:property name="wheel_mass"   value="8.0"/>
   <xacro:property name="wheel_radius" value="0.16459"/>
   <xacro:property name="wheel_length" value="0.11653"/>
-  <xacro:property name="wheel_mass" value="8"/>
   <xacro:property name="wheel_offset_x" value="0.249"/>
   <xacro:property name="wheel_offset_y" value="0.29153"/>
   <xacro:property name="wheel_offset_z" value="-0.0702"/>
-  <xacro:property name="camera_size" value="0.02"/>
-  <xacro:property name="lidar_radius" value="0.03"/>
-  <xacro:property name="lidar_length" value="0.1"/>
-  <!-- 계산된 속성
-  <xacro:property name="wheel_separation" value="${wheel_offset_y * 2}"/>
-  -->
-  <!-- 재질 정의 -->
+  <xacro:property name="camera_size"   value="0.02"/>
+  <xacro:property name="lidar_radius"  value="0.03"/>
+  <xacro:property name="lidar_length"  value="0.1"/>
   <material name="red"><color rgba="1.0 0.0 0.0 1.0"/></material>
   <material name="black"><color rgba="0 0 0 1"/></material>
-  <!-- 바퀴 매크로 정의 -->
-  <xacro:macro name="wheel" params="prefix pos_x pos_y pos_z flip wheel_type *origin *axis">
+  <xacro:macro name="wheel" params="prefix wheel_type *origin *axis">
     <link name="${prefix}_wheel_link">
       <visual>
@@ -30,13 +23,13 @@
       </visual>
       <collision>
-        <origin rpy="1.570795 0 0"/>
+        <origin rpy="1.570795 0 0" xyz="0 0 0"/>
         <geometry><cylinder length="${wheel_length}" radius="${wheel_radius}"/></geometry>
       </collision>
       <inertial>
+        <origin xyz="0 0 0" rpy="0 0 0"/>
         <mass value="${wheel_mass}"/>
         <inertia ixx="${(1/12) * wheel_mass * (3*wheel_radius*wheel_radius + wheel_length*wheel_length)}" ixy="0" ixz="0"
                  iyy="${(1/12) * wheel_mass * (3*wheel_radius*wheel_radius + wheel_length*wheel_length)}" iyz="0"
                  izz="${(1/2) * wheel_mass * (wheel_radius*wheel_radius)}"/>
-        <!-- <inertia ixx="0.1171" ixy="0" ixz="0" iyy="0.1361" iyz="0" izz="0.1171"/> -->
       </inertial>
     </link>
@@ -49,27 +42,23 @@
       <dynamics damping="0.0" friction="20"/>
     </joint>
-    <!-- Gazebo 속성 적용 -->
     <xacro:wheel_gazebo prefix="${prefix}"/>
   </xacro:macro>
-  <!-- 바퀴 생성 -->
-  <xacro:wheel prefix="front_right" pos_x="${wheel_offset_x}" pos_y="${-wheel_offset_y}" pos_z="${wheel_offset_z}" flip="true" wheel_type="wheel_type1">
+  <xacro:wheel prefix="front_right" wheel_type="wheel_type1">
     <origin rpy="3.14 0 0" xyz="${wheel_offset_x} ${-wheel_offset_y} ${wheel_offset_z}"/>
     <axis xyz="0 -1 0"/>
   </xacro:wheel>
-  <xacro:wheel prefix="front_left" pos_x="${wheel_offset_x}" pos_y="${wheel_offset_y}" pos_z="${wheel_offset_z}" flip="false" wheel_type="wheel_type2">
+  <xacro:wheel prefix="front_left" wheel_type="wheel_type2">
     <origin rpy="0 0 0" xyz="${wheel_offset_x} ${wheel_offset_y} ${wheel_offset_z}"/>
     <axis xyz="0 1 0"/>
   </xacro:wheel>
-  <xacro:wheel prefix="rear_left" pos_x="${-wheel_offset_x}" pos_y="${wheel_offset_y}" pos_z="${wheel_offset_z}" flip="false" wheel_type="wheel_type2">
+  <xacro:wheel prefix="rear_left" wheel_type="wheel_type2">
     <origin rpy="0 0 0" xyz="${-wheel_offset_x} ${wheel_offset_y} ${wheel_offset_z}"/>
     <axis xyz="0 1 0"/>
   </xacro:wheel>
-  <xacro:wheel prefix="rear_right" pos_x="${-wheel_offset_x}" pos_y="${-wheel_offset_y}" pos_z="${wheel_offset_z}" flip="true" wheel_type="wheel_type1">
+  <xacro:wheel prefix="rear_right" wheel_type="wheel_type1">
     <origin rpy="3.14 0 0" xyz="${-wheel_offset_x} ${-wheel_offset_y} ${wheel_offset_z}"/>
     <axis xyz="0 -1 0"/>
   </xacro:wheel>
-  <!-- Base footprint link -->
   <link name="base_footprint"/>
-  <!-- Base link -->
   <link name="base_link">
     <visual>
@@ -79,20 +68,16 @@
     <collision>
       <origin xyz="0 0 0.008"/>
-      <geometry><box size="${base_length} ${base_width} ${base_height}"/>
-      </geometry>
+      <geometry><box size="${base_length} ${base_width} ${base_height}"/></geometry>
     </collision>
     <collision>
       <origin xyz="0 0 0.035"/>
-      <geometry>
-        <box size="0.154 0.627 0.07"/>
-      </geometry>
+      <geometry><box size="0.154 0.627 0.07"/></geometry>
     </collision>
     <inertial>
-      <mass value="50"/>
+      <mass value="${base_mass}"/>
       <origin xyz="0.0 0.0 0.015"/>
-      <!-- <inertia ixx="2.288641" ixy="0" ixz="0" iyy="5.103976" iyz="0" izz="3.431465"/></inertial> -->
-      <inertia ixx="${(1/12) * 50 * (base_width*base_width + base_height*base_height)}" ixy="0" ixz="0"
-             iyy="${(1/12) * 50 * (base_length*base_length + base_height*base_height)}" iyz="0"
-             izz="${(1/12) * 50 * (base_length*base_length + base_width*base_width)}"/>
+      <inertia ixx="${(1/12) * base_mass * (base_width*base_width + base_height*base_height)}" ixy="0" ixz="0"
+               iyy="${(1/12) * base_mass * (base_length*base_length + base_height*base_height)}" iyz="0"
+               izz="${(1/12) * base_mass * (base_length*base_length + base_width*base_width)}"/>
     </inertial>
   </link>
@@ -102,55 +87,39 @@
     <origin xyz="0 0 0.2352" rpy="0 0 0"/>
   </joint>
-  <!-- Camera link -->
   <link name="camera_link">
     <visual>
-      <geometry>
-        <box size="${camera_size} ${camera_size} ${camera_size}"/>
-      </geometry>
+      <geometry><box size="${camera_size} ${camera_size} ${camera_size}"/></geometry>
       <material name="red"/>
     </visual>
     <collision>
-      <geometry>
-        <box size="${camera_size} ${camera_size} ${camera_size}"/>
-      </geometry>
+      <geometry><box size="${camera_size} ${camera_size} ${camera_size}"/></geometry>
     </collision>
     <inertial>
       <mass value="0.1"/>
-      <!-- <inertia ixx="0.000083" ixy="0" ixz="0" iyy="0.000083" iyz="0" izz="0.000083"/></inertial> -->
       <inertia ixx="${(1/12) * 0.1 * (camera_size*camera_size + camera_size*camera_size)}" ixy="0" ixz="0"
-             iyy="${(1/12) * 0.1 * (camera_size*camera_size + camera_size*camera_size)}" iyz="0"
-             izz="${(1/12) * 0.1 * (camera_size*camera_size + camera_size*camera_size)}"/>
+               iyy="${(1/12) * 0.1 * (camera_size*camera_size + camera_size*camera_size)}" iyz="0"
+               izz="${(1/12) * 0.1 * (camera_size*camera_size + camera_size*camera_size)}"/>
     </inertial>
   </link>
   <joint name="camera_joint" type="fixed">
-    <parent link="base_link"/>
-    <child link="camera_link"/>
-    <origin xyz="0.40 0.0 0.04"/>
+    <parent link="base_link"/><child link="camera_link"/><origin xyz="0.40 0.0 0.04"/>
   </joint>
-  <!-- 2D LiDAR Link -->
   <link name="lidar_link">
     <visual>
-      <geometry>
-        <cylinder radius="${lidar_radius}" length="${lidar_length}"/>
-      </geometry>
+      <geometry><cylinder radius="${lidar_radius}" length="${lidar_length}"/></geometry>
       <material name="black"/>
     </visual>
     <collision>
-      <geometry>
-        <cylinder radius="${lidar_radius}" length="${lidar_length}"/>
-      </geometry>
+      <geometry><cylinder radius="${lidar_radius}" length="${lidar_length}"/></geometry>
     </collision>
     <inertial>
       <mass value="0.1"/>
-      <!-- <inertia ixx="0.000045" ixy="0" ixz="0" iyy="0.000045" iyz="0" izz="0.000075"/></inertial> -->
       <inertia ixx="${(1/12) * 0.1 * (3*lidar_radius*lidar_radius + lidar_length*lidar_length)}" ixy="0" ixz="0"
-                 iyy="${(1/12) * 0.1 * (3*lidar_radius*lidar_radius + lidar_length*lidar_length)}" iyz="0"
-                 izz="${(1/2) * 0.1 * (lidar_radius*lidar_radius)}"/>
-      </inertial>
+               iyy="${(1/12) * 0.1 * (3*lidar_radius*lidar_radius + lidar_length*lidar_length)}" iyz="0"
+               izz="${(1/2) * 0.1 * lidar_radius*lidar_radius}"/>
+    </inertial>
   </link>
   <joint name="lidar_joint" type="fixed">
-    <parent link="base_link"/>
-    <child link="lidar_link"/>
-    <origin xyz="0 0 0.13" rpy="0 0 0"/>
+    <parent link="base_link"/><child link="lidar_link"/><origin xyz="0 0 0.13" rpy="0 0 0"/>
   </joint>
 </robot>
