Commit message: new boxbot URDF

File: src/my_box_bot_description/urdf/box_bot.urdf (robot description, URDF)
Before this commit: robot box_bot, 10 links, 9 joints
Links:
- removed link chassis
- removed link left_wheel
- removed link right_wheel
- added link base_footprint
- added link left_wheel_link, mass 0.05; collision cylinder length=0.001 radius=0.035; visual cylinder length=0.01 radius=0.035
- added link right_wheel_link, mass 0.05; collision cylinder length=0.001 radius=0.035; visual cylinder length=0.01 radius=0.035
- link back_roll_link: geometry collision cylinder length=0.001 radius=0.0045; visual cylinder length=0.005 radius=0.010
- link back_yaw_link: geometry collision cylinder length=0.001 radius=0.0045; visual cylinder length=0.005 radius=0.010
- link base_link: mass None -> 0.5; geometry collision box size=0.1 0.1 0.1; visual mesh filename=package://my_box_bot_description/meshes/cute_cube.dae scale=0.1 0.1 0.1
- link front_roll_link: geometry collision cylinder length=0.001 radius=0.0045; visual cylinder length=0.005 radius=0.010
- link front_yaw_link: geometry collision cylinder length=0.001 radius=0.0045; visual cylinder length=0.005 radius=0.010
Joints:
- removed joint joint_left_wheel
- removed joint joint_right_wheel
- added joint left_wheel_joint: type continuous, parent base_link, child left_wheel_link, origin xyz=0 0.05 -0.025 rpy=0 0 0, axis 0 1 0, limit effort=10000 velocity=1000
- added joint right_wheel_joint: type continuous, parent base_link, child right_wheel_link, origin xyz=0 -0.05 -0.025 rpy=0 0 0, axis 0 1 0, limit effort=10000 velocity=1000
- joint back_yaw_joint: parent chassis -> base_link
- joint base_link_joint: child chassis -> base_link; origin xyz=0 0 0 rpy=0 0 0 -> xyz=0 0 0.0175 rpy=0 0 0; parent base_link -> base_footprint
- joint front_yaw_joint: parent chassis -> base_link

File: src/urdfbot_description/urdf/urdfbot_simple2.urdf (robot description, URDF)
Before this commit: robot urdfbot, 6 links, 5 joints
Joints:
- joint base_link_to_head_link_joint: origin xyz=0 0 0.07 rpy=0 0 0 -> xyz=0 0 0.06 rpy=0 0 0
