Commit message: add 라이더 및 imu 센서 추가

File: src/my_box_bot_description/urdf/box_bot3.urdf (robot description, URDF)
Before this commit: robot box_bot, 7 links, 6 joints
Links:
- added link laser_scan_link, mass 0.01; collision cylinder length=0.0408 radius=0.037493; visual mesh filename=package://my_box_bot_description/meshes/sensors/rplidar.dae scale=1.0 1.0 1.0
- link imu_link: geometry visual box size=0.015 0.015 0.0025
Joints:
- added joint laser_scan_link_joint: type continuous, parent base_link, child laser_scan_link, origin xyz=0 0 0.05 rpy=0 0 0, axis 0 0 1, limit effort=10.0 velocity=100.0
- joint imu_joint: origin xyz=0.03 0.03 0.05 rpy=0 0 0 -> xyz=0.037 0.037 0.051 rpy=0 0 0
