Commit message: add 4/17

File: src/my_box_bot_description/urdf/box_bot2.urdf (robot description, URDF)
Before this commit: robot box_bot, 7 links, 6 joints
Links:
- link imu_link: geometry visual box size=0.015 0.015 0.0025
Joints:
- joint imu_joint: origin xyz=0.03 0.03 0.05 rpy=0 0 0 -> xyz=0.037 0.037 0.051 rpy=0 0 0

File: src/my_box_bot_description/urdf/box_bot3.urdf (robot description, URDF)
Before this commit: robot box_bot, 8 links, 7 joints
Links:
- added link camera_link, mass 0.1; collision box size=0.04 0.17 0.03; visual mesh filename=package://my_box_bot_description/meshes/sensors/realsense.d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 scale=1.0 1.0 1.0
Joints:
- added joint camera_link_joint: type fixed, parent base_link, child camera_link, origin xyz=0.08 0 0.06 rpy=0 -0.2 0
